Commit message: [Fix]: isr_m4.urdf.xacro: fixed the path to the stl file

File: isr_m4_description/urdf/isr_m4.urdf.xacro (robot description, xacro)
@@ -6,5 +6,5 @@
       <origin xyz="0 0 0.457" rpy="-1.57 0 -1.57" />
       <geometry>
-        <mesh filename="package://isr_m4_description/meshes/isr_m3.stl" scale="0.001 0.001 0.001" />
+        <mesh filename="file://$(find isr_m4_description)/meshes/isr_m3.stl" scale="0.001 0.001 0.001" />
       </geometry>
       <material name="light_black">
